File: hardware/BREAD_Slice.kicad_sch (KiCad schematic)
At the start: 15 parts, among them J1 I2C_01x04, J2 Conn_01x10_Female

Commit message: feat(hw): redesign charger stage from the BQ24650 reference design
Rebuild the charger sheet against the BQ24650 datasheet and the
BQ24650EVM-639 reference design: PDS1040-13 and ZLLS350TA Schottky
diodes, SI7288DP-T1-GE3 dual MOSFET, input and output filtering, and
test points per the EVM. Every symbol now resolves from
KiCad-Master-Lib; the *-rescue, kml-custom and SparkFun references are
gone, and the top sheet drops the unused I2C header.

The bootstrap diode is oriented REGN -> BTST as the datasheet requires,
and the BQ24650 VCC net carries a PWR_FLAG since it is fed through the
input filter resistors. ERC is clean at all severities.

The PCB is cleared for re-layout: the Nano socket, buck stage and
mechanicals are placed, nothing is routed, and DRC schematic parity
reports 66 missing footprints until layout lands.
Parts:
- removed J1: I2C_01x04, Connector_JST:JST_SH_SM04B-SRSS-TB_1x04-1MP_P1.00mm_Horizontal, symbol SparkFun-Connector:I2C_01x04
- D1: symbol SparkFun-LED:WS2812B_5050 -> KMLib_IC_Digital:WS2812B_5050_RGB_LED; PROD_ID (none) -> DIO-12503
- J1: renamed from J2; symbol Connector:Conn_01x10_Female -> Connector:Conn_01x10_Socket
- U1: value (none) -> AP63205WU-7; footprint Package_TO_SOT_SMD:TSOT-23-6 -> KMLib_IC_SMD:SOIC_05WU-7_DIO
Connections:
- net STAT1_IN: now also A1.21 (A2); no longer A1.20 (A1)
- net STAT2_IN: now also A1.20 (A1); no longer A1.21 (A2)
Other:
- sheet BQ24650 Solar Charger ports: added none; removed VCC
