File: hardware/Solar-Battery-Charger.kicad_sch (KiCad schematic)
At the start: 48 parts, among them J3 Conn_01x02_Female, J4 Tab_Amp_1217861-1, J5 Tab_Amp_1217861-1, J6 Tab_Amp_1217861-1, J7 Tab_Amp_1217861-1, Q1 AO4882, Q2 2N7002, U2 LM234Z-3, U3 NSL-32, U4 BQ24650RVAT, U5 NSL-32

Commit message: chore(hw): migrate KiCad files to the KiCad 10 format
Via `kicad-cli sch upgrade` / `pcb upgrade` (bread-infra
scripts/upgrade_kicad10.sh). Verified lossless: identical netlist, footprint
positions and routing.

Note `sch upgrade` does not cascade into hierarchical sub-sheets, so every
.kicad_sch is upgraded individually -- upgrading only the root sheet leaves
sub-sheets on the old format, which looks migrated and is not.
Parts:
- R7: value 80m - sense res -> 80m - sense res

Commit message: fix(hw): re-point stale library nicknames
These parts exist in KiCad-Master-Lib; the boards referenced libraries that no
longer exist (kml-custom, KML-Custom, and SparkFun libraries that never
contained the part) or names the library has since changed.

KiCad embeds footprint geometry in the .kicad_pcb, so the boards rendered and
fabricated correctly and the rot stayed invisible -- it only surfaces on
update-from-library, or when a generator tries to resolve a nickname.

Nickname/name only. No geometry is changed:

  KML-Custom:CDBA-G -> KMLib_Passives_SMD:CDBA-G
  KML-Custom:RVA16_2P14X2P14 -> KMLib_IC_SMD:RVA16_2P14X2P14
  KML-Custom:Thermal Pad -> KMLib_Mounting:Thermal_Pad
  SparkFun-DiscreteSemi:AP63205 -> KMLib_IC_Power:AP63205WU-7_Buck_Regulator
  SparkFun-Fuse:Thermal Pad -> KMLib_Mounting:Thermal_Pad
  SparkFun-LED:WS2812-5050-4PIN -> KMLib_IC_SMD:WS2812-5050-4PIN
  kml-custom:BQ24650RVAT -> KMLib_IC_Power:BQ24650RVAT_Charger_Controller

Only references that failed to resolve were touched. Generic parts (<=4 pins)
and KiCad *-rescue libraries are deliberately excluded: fingerprint matching
cannot distinguish a 2-pin resistor from a 2-pin capacitor, so those are being
done by hand.
Parts:
- D3: footprint KML-Custom:CDBA-G -> KMLib_Passives_SMD:CDBA-G
- U4: footprint KML-Custom:RVA16_2P14X2P14 -> KMLib_IC_SMD:RVA16_2P14X2P14; symbol kml-custom:BQ24650RVAT -> KMLib_IC_Power:BQ24650RVAT_Charger_Controller
Changed lines of the file:
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@@
 	)
 	(symbol
-		(lib_id "kml-custom:BQ24650RVAT")
+		(lib_id "KMLib_IC_Power:BQ24650RVAT_Charger_Controller")
 		(at 177.8 93.98 0)
 		(unit 1)
@@
 			)
 		)
-		(property "Footprint" "KML-Custom:RVA16_2P14X2P14"
+		(property "Footprint" "KMLib_IC_SMD:RVA16_2P14X2P14"
 			(at 177.8 93.98 0)
 			(hide yes)
@@
 			)
 		)
-		(property "Footprint" "KML-Custom:CDBA-G"
+		(property "Footprint" "KMLib_Passives_SMD:CDBA-G"
 			(at 52.07 21.59 0)
 			(hide yes)
